File: MCU.brd (EAGLE design)
At the start: 69.5 x 25.5 mm, 46 parts, among them CN2 JSTPH, IC1 MEGA328-A, IC2 L4931D, Q1-M 8MHz, 22pF, U2 MCP73831T-2ACI/OT, U3 FTS31XS-U

Commit message: Add files via upload
Parts:
- removed C10-R, C14-U, C6-PB: 0.1uF, SparkFun-Capacitors:0603-CAP
- removed C11-R: 2.2uF, SparkFun-Capacitors:0603-CAP
- removed C12-U, C13-U: 47pF, SparkFun-Capacitors:0603-CAP
- removed C4-PB, C8-C, C9-C: 10µF, microbuilder:0805-NO
- removed C7-PB: 1uF, SparkFun-Capacitors:0603-CAP
- removed CN2: JSTPH, microbuilder:JSTPH2
- removed D1-PB: 1N4004, diode:DO41-10
- removed IC2: L4931D, v-reg-3:SO08
- removed JP2: USB-MICROB", SparkFun-Connectors:USB-B-MICRO-SMD_V03
- removed LED1-R, LED3-C: RED, microbuilder:CHIPLED_0805_NOOUTLINE
- removed LED4-C: GREEN, microbuilder:CHIPLED_0805_NOOUTLINE
- removed N_FET, P_FET: (no value), transistor-fet:TO92
- removed ON/OFF: DTE6K, switch-misc:DTE6K
- removed R10-C: 5K\, microbuilder:0805-NO
- removed R12-R: 330, microbuilder:0805-NO
- removed R13-U, R14-U: 27, SparkFun-Resistors:0603-RES
- removed R4-PB, R7-PB: 100k, rcl:R0805
- removed R5-PB: 300k, rcl:R0805
- removed R6-PB: 10k, rcl:R0805
- removed R8-C, R9-C: 470, microbuilder:0805-NO
- removed U2: MCP73831T-2ACI/OT, microbuilder:SOT23-5
- removed U3: FTS31XS-U, SparkFun-DigitalIC:SSOP20_L
- RESET: value DTE6K -> (none); device switch-misc:DTE6K -> switch-omron:B3F-10XX
- moved IC1 83.6 mm to (0.50, -66.0)
- moved Q1-M 74.0 mm to (17.5, -62.0), turned to 0 degrees
- moved R6-PB1 69.5 mm to (9.00, -63.0)
- moved C2-M 68.5 mm to (23.0, -61.0)
- moved FLX0- 66.7 mm to (2.00, -51.5)
- moved ACC_X 61.4 mm to (2.00, -35.0)
- moved FLX1- 57.3 mm to (18.5, -51.5)
- moved RESET 56.0 mm to (5.00, -17.0)
- moved FLX2- 54.0 mm to (35.0, -51.5)
- moved ACC_Y 47.4 mm to (18.5, -35.0)
- moved GND_PAD 43.9 mm to (40.5, -16.0), turned to 0 degrees
- moved VCC_PAD 39.7 mm to (46.0, -16.0), turned to 0 degrees
- moved ACC_Z 38.7 mm to (35.0, -35.0)
- moved JP1 19.4 mm to (26.5, -16.0)
Connections:
- removed net CBUS0: U3.18
- removed net CBUS3: U3.19
- removed net CTS: U3.9
- removed net DCD: U3.8
- removed net DSR: U3.7
- removed net N$1: R13-U.2, U3.12
- removed net N$11: R14-U.1, U3.11
- removed net N$12: C12-U.1, JP2.D+1, R14-U.2
- removed net N$15: C6-PB.2, C7-PB.2, N_FET.3, P_FET.1, R7-PB.2
- removed net N$16: LED3-C.C, R8-C.1
- removed net N$17: R8-C.2, R9-C.2, U2.1
- removed net N$18: R10-C.1, U2.5
- removed net N$19: LED4-C.A, R9-C.1
- removed net N$21: C13-U.1, JP2.D-1, R13-U.1
- removed net N$22: U3.17
- removed net N$23: U3.10
- removed net N$5: C7-PB.1, D1-PB.C, ON/OFF.1, ON/OFF.2, R6-PB.2
- removed net N$7: LED1-R.A, R12-R.2
- removed net N$9: C4-PB.2, N_FET.2, R5-PB.1
- removed net RI: U3.5
- removed net RTS: U3.2
- removed net VBAT: C6-PB.1, C9-C.1, CN2.2, P_FET.3, R6-PB.1, R7-PB.1, U2.3
- removed net VBUS: C8-C.1, JP2.VBUS1, LED3-C.A, U2.4
- removed net V_IN: C10-R.1, C4-PB.1, IC2.8, P_FET.2, R4-PB.1
- net 3.3V: no longer C11-R.1, C14-U.1, IC2.1, R12-R.1, U3.13, U3.14, U3.15, U3.3
- net DTR: no longer U3.1
- net GND: no longer C10-R.2, C11-R.2, C12-U.2, C13-U.2, C14-U.2, C8-C.2, C9-C.2, CN2.1, IC2.2, JP2.GND1, JP2.SHIELD1, JP2.SHIELD2, JP2.SHIELD3, LED1-R.C, LED4-C.C, N_FET.1, ON/OFF.3, ON/OFF.4, R10-C.2, U2.2, U3.16, U3.6
- net POWER_OFF: no longer D1-PB.A, R4-PB.2, R5-PB.2
- net RXI: no longer U3.4
- net TXO: no longer U3.20
Routing:
- net GND: track 201.5 -> 0.00 mm, vias 3 -> 0
- net 3.3V: track 132.3 -> 0.00 mm, vias 4 -> 0
- net VBAT: track 92.7 -> 0.00 mm, vias 5 -> 0
- net N$12: track 52.6 -> 0.00 mm, vias 3 -> 0
- net N$2: track 45.3 -> 0.00 mm, vias 1 -> 0
- net POWER_OFF: track 44.5 -> 0.00 mm, vias 3 -> 0
- net DTR: track 37.3 -> 0.00 mm, vias 2 -> 0
- net N$5: track 35.7 -> 0.00 mm
- net V_IN: track 34.7 -> 0.00 mm
- net N$11: track 30.4 -> 0.00 mm, vias 2 -> 0
- net TXO: track 29.7 -> 0.00 mm, vias 4 -> 0
- net N$1: track 25.7 -> 0.00 mm
- net N$17: track 25.2 -> 0.00 mm, vias 2 -> 0
- net N$15: track 19.7 -> 0.00 mm
- net RXI: track 18.2 -> 0.00 mm, vias 2 -> 0
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- removed copper zone on layer 1, net N$6
- removed copper zone on layer 16, net N$8
Other:
- board size 69.5 x 25.5 mm -> 47.5 x 21.5 mm
