File: MCU.sch (EAGLE design)
At the start: 46 parts, among them CN2 JSTPH, IC1 MEGA328-A, IC2 L4931D, Q1-M 8MHz, 22pF, U2 MCP73831T-2ACI/OT, U3 FTS31XS-U

Commit message: Add files via upload
Parts:
- removed C10-R, C14-U, C6-PB: 0.1uF, SparkFun-Capacitors:0.1UF-25V(+80/-20%)(0603)
- removed C11-R: 2.2uF, SparkFun-Capacitors:0.1UF-25V(+80/-20%)(0603)
- removed C12-U, C13-U: 47pF, SparkFun-Capacitors:47PF-50V-5%(0603)
- removed C4-PB, C8-C, C9-C: 10µF, microbuilder:CAP_CERAMIC0805-NOOUTLINE
- removed C7-PB: 1uF, SparkFun-Capacitors:0.1UF-25V(+80/-20%)(0603)
- removed CN2: JSTPH, microbuilder:JST_2PIN
- removed D1-PB: 1N4004, diode:1N4004
- removed IC2: L4931D, v-reg-3:L4931D
- removed JP2: USB-MICROB", SparkFun-Connectors:USB-MICROB"
- removed LED1-R, LED3-C: RED, microbuilder:LED0805_NOOUTLINE
- removed LED4-C: GREEN, microbuilder:LED0805_NOOUTLINE
- removed N_FET: BSS101, transistor-fet:BSS101
- removed ON/OFF: DTE6K, switch-misc:DTE6K
- removed P_FET: BSS92, transistor-fet:BSS92
- removed R10-C: 5K\, microbuilder:RESISTOR0805_NOOUTLINE
- removed R12-R: 330, microbuilder:RESISTOR0805_NOOUTLINE
- removed R13-U, R14-U: 27, SparkFun-Resistors:27OHM1/10W1%(0603)0603-RES
- removed R4-PB, R7-PB: 100k, rcl:R-US_R0805
- removed R5-PB: 300k, rcl:R-US_R0805
- removed R6-PB: 10k, rcl:R-US_R0805
- removed R8-C, R9-C: 470, microbuilder:RESISTOR0805_NOOUTLINE
- removed U2: MCP73831T-2ACI/OT, microbuilder:MCP73831/2
- removed U3: FTS31XS-U, SparkFun-DigitalIC:FT231XS
- RESET: value DTE6K -> (none); device switch-misc:DTE6K -> switch-omron:10-XX
Connections:
- removed net CBUS0: U3.CBUS0
- removed net CBUS3: U3.CBUS3
- removed net CTS: U3.!CTS
- removed net DCD: U3.!DCD
- removed net DSR: U3.!DSR
- removed net N$1: R13-U.2, U3.USBDM
- removed net N$11: R14-U.1, U3.USBDP
- removed net N$12: C12-U.1, JP2.D+, R14-U.2
- removed net N$15: C6-PB.2, C7-PB.2, N_FET.D, P_FET.G, R7-PB.2
- removed net N$16: LED3-C.C, R8-C.1
- removed net N$17: R8-C.2, R9-C.2, U2.STAT
- removed net N$18: R10-C.1, U2.PROG
- removed net N$19: LED4-C.A, R9-C.1
- removed net N$21: C13-U.1, JP2.D-, R13-U.1
- removed net N$22: U3.CBUS1
- removed net N$23: U3.CBUS2
- removed net N$5: C7-PB.1, D1-PB.C, ON/OFF.S, ON/OFF.S@1, R6-PB.2
- removed net N$7: LED1-R.A, R12-R.2
- removed net N$9: C4-PB.2, N_FET.G, R5-PB.1
- removed net RI: U3.!RI
- removed net RTS: U3.!RTS
- removed net VBAT: C6-PB.1, C9-C.1, CN2.2, P_FET.S, R6-PB.1, R7-PB.1, U2.VBAT
- removed net VBUS: C8-C.1, JP2.VBUS, LED3-C.A, U2.VDD
- removed net V_IN: C10-R.1, C4-PB.1, IC2.VIN, P_FET.D, R4-PB.1
- net 3.3V: no longer C11-R.1, C14-U.1, IC2.VOUT, R12-R.1, U3.!RESET, U3.3V3OUT, U3.VCC, U3.VCCIO
- net DTR: no longer U3.!DTR
- net GND: now also RESET.P1; no longer C10-R.2, C11-R.2, C12-U.2, C13-U.2, C14-U.2, C8-C.2, C9-C.2, CN2.1, IC2.GND, JP2.GND, JP2.SHIELD, LED1-R.C, LED4-C.C, N_FET.S, ON/OFF.P, ON/OFF.P@1, R10-C.2, RESET.P@1, U2.VSS, U3.GND@16, U3.GND@6
- net N$2: now also RESET.S1; no longer RESET.S@1
- net POWER_OFF: no longer D1-PB.A, R4-PB.2, R5-PB.2
- net RXI: no longer U3.RXD
- net TXO: no longer U3.TXD
Other:
- note removed: "1.0K = 1000mA"
- note removed: "10K = 100mA"
- note removed: "2.0K = 500mA"
- note removed: "5.0K = 200mA"
- note removed: "Connections needed for communications are TXD, RXD, & GND. 3.3V is internally regulated"
- note removed: "Micro USB Lipo Charger"
- note removed: "Push Button Power Circuit"
- note removed: "USB to UART Serial Module"
- note removed: "Very Low Dropout Voltage Regulator"
- moved on the sheet: ACC_X, ACC_Y, ACC_Z, C2-M, FLX0-, FLX1-, FLX2-, GND_PAD, IC1, JP1, Q1-M, R6-PB1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
