File: Full System.sch (EAGLE design)
At the start: 46 parts, among them CN2 JSTPH, IC1 MEGA328-A, IC2 L4931D, Q1-M 8MHz, 22pF, U2 MCP73831T-2ACI/OT, U3 FTS31XS-U

Commit message: Add files via upload
Parts:
- removed ON/OFF, RESET: (no value), switch-omron:10-XX
- added C1: 0.1uF, SparkFun:CAP0603-CAP
- added C2: 10uF, SparkFun:CAP_POL1206
- added LED2-M: Blue, microbuilder:LED0805_NOOUTLINE
- added R1-M1, R1-M2, R1-M3, R2-M, R2-M1, R3-M: 10k, rcl:R-US_R0805
- added S1: Power, Spark:TAC_SWITCHSMD
- added S2: Option, Spark:TAC_SWITCHSMD
- added S3: BT_C, Spark:TAC_SWITCHSMD
- added U1: BLUETOOTH-RN41", SparkFun-RF:BLUETOOTH-RN41"
- D1-PB: value 1N4004 -> (none); device diode:1N4004 -> semicon-smd-ipc:D-A1-C3
- renumbered R6-PB1 to R1-M
Connections:
- removed net FLX!: IC1.PC1(ADC1)
- removed net N$13: IC1.PB0(ICP)
- removed net N$14: IC1.PB1(OC1A)
- new net FLX1: FLX1-.P, IC1.PC1(ADC1), R1-M2.1
- new net LED1: IC1.PB0(ICP), R2-M1.1
- new net N$10: LED2-M.C, R2-M1.2
- new net N$6: IC1.PD4(XCK/T0), R3-M.1, S3.1
- new net PIO10: U1.PIO10
- new net PIO11: U1.PIO11
- new net PIO2: U1.PIO2
- new net PIO3: U1.PIO3
- new net PIO4: U1.PIO4
- new net PIO5: U1.PIO5
- new net PIO6: U1.PIO6
- new net PIO7: U1.PIO7
- new net RESET: C2-M.1, IC1.PC6(/RESET), R1-M.2, U1.RESET
- new net SPICLK: U1.SPICLK
- new net SPICSB: U1.SPICSB
- new net SPIMISO: U1.SPIMISO
- new net SPIMOSI: U1.SPIMOSI
- new net UARTCTS: U1.UARTCTS
- new net UARTRTS: U1.UARTRTS
- new net UARTRX: U1.UARTRX
- new net UARTTX: U1.UARTTX
- net 3.3V: now also LED2-M.A, R2-M.2, R3-M.2
- net ACC_X: now also ACC_X.P
- net ACC_Y: now also ACC_Y.P
- net ACC_Z: now also ACC_Z.P
- net FLX0: now also FLX0-.P, R1-M1.1
- net FLX2: now also FLX2-.P, R1-M3.1
- net GND: now also C1.2, C2.-, R1-M1.2, R1-M2.2, R1-M3.2, S1.2, S2.3, S3.3, U1.GND, U1.GND1, U1.GND2, U1.GND3; no longer ON/OFF.P, ON/OFF.P1, Q1-M.2, RESET.P, RESET.P1
- net N$2: now also IC1.PD3(INT1), R2-M.1, S2.1; no longer C2-M.1, IC1.PC6(/RESET), R1-M.2, RESET.S, RESET.S1
- net N$3: no longer Q1-M.1
- net N$4: no longer Q1-M.3
- net N$5: now also S1.4; no longer ON/OFF.S, ON/OFF.S1
- net VCC: now also C1.1, C2.+, U1.VDD
Other:
- moved on the sheet: FLX0-, FLX1-, FLX2-, GND_PAD, VCC_PAD
